Commit message: add floating joint of robot base in model

File: ros/src/teleop_motorhand/robots/tams_motorhand.urdf.xacro (robot description, xacro)
@@ -14,4 +14,8 @@
     <origin xyz="0.0 0.0 0.0" rpy="0.0 0.0 0.0" />
   </joint>
+  <!-- <joint name="rh_world_joint" type="floating">
+    <parent link="world" />
+    <child link="rh_forearm" />
+  </joint> -->
   <xacro:tams_motorhand prefix="rh_" />
 </robot>
